Commit message: set caster wheel to box collision

File: robots/donatello/urdf/robot.xacro (robot description, xacro)
@@ -52,5 +52,5 @@
     <origin xyz="${casterRadius-chassisLength/2} 0 ${casterRadius-chassisHeight+wheelRadius}" rpy="0 0 0"/>
     <geometry>
-      <sphere radius="${casterRadius}"/>
+      <box size="${casterRadius*2} ${casterRadius*2} ${casterRadius*2}"/>
     </geometry>
   </collision>
@@ -65,4 +65,5 @@
     <origin xyz="${casterRadius-chassisLength/2} 0 ${casterRadius-chassisHeight+wheelRadius}" rpy="0 0 0"/>
     <mass value="${casterMass}"/>
+    <box_inertia m="${casterMass}" x="${casterRadius*2}" y="${casterRadius*2}" z="${casterRadius*2}"/>
     <sphere_inertia m="${casterMass}" r="${casterRadius}"/>
   </inertial>
