Commit message: add wheel model

File: robots/donatello/urdf/macros.xacro (robot description, xacro)
@@ -28,9 +28,9 @@
   </collision>
   <visual>
-    <origin xyz="0 0 0" rpy="0 ${PI/2} ${PI/2}" />
+    <origin xyz="0 0 0" rpy="0 0 0" />
     <geometry>
-      <cylinder length="${wheelWidth}" radius="${wheelRadius}"/>
+      <mesh filename="package://roberta_sim/robots/donatello/meshes/${lr}_tire.stl" scale="${wheelRadius*0.001/0.033} ${0.001*wheelWidth/0.018} ${0.001*wheelRadius/0.033}"/>
     </geometry>
-    <material name="black"/>
+    <material name="dark"/>
   </visual>
   <inertial>
@@ -46,5 +46,5 @@
   <kd  value="1.0" />
   <fdir1 value="1 0 0"/>
-  <material>Gazebo/Black</material>
+  <material>Gazebo/FlatBlack</material>
 </gazebo>
 <joint name="${lr}_wheel_joint" type="continuous">

Commit message: add  roberta map und dif control

File: robots/donatello/urdf/macros.xacro (robot description, xacro)
@@ -41,9 +41,11 @@
 </link>
 <gazebo reference="${lr}_wheel">
-  <mu1 value="1.0"/>
-  <mu2 value="1.0"/>
-  <kp  value="10000000.0" />
-  <kd  value="1.0" />
-  <fdir1 value="1 0 0"/>
+    <mu1>0.1</mu1>
+    <mu2>0.1</mu2>
+    <kp>500000.0</kp>
+    <kd>10.0</kd>
+    <minDepth>0.001</minDepth>
+    <maxVel>0.1</maxVel>
+    <fdir1>1 0 0</fdir1>
   <material>Gazebo/FlatBlack</material>
 </gazebo>
@@ -53,8 +55,8 @@
   <origin xyz="${chassisLength/2-wheelPos} ${tY*wheelWidth/2+tY*chassisWidth/2} ${wheelRadius}" rpy="0 0 0" />
   <axis xyz="0 1 0" rpy="0 0 0" />
-  <limit effort="100" velocity="100"/>
-  <dynamics damping="0.0" friction="0.0"/>
+  <!--limit effort="100" velocity="100"/>
+  <dynamics damping="0.0" friction="0.0"/-->
 </joint>
-<transmission name="${lr}_wheel_trans">
+<!--transmission name="${lr}_wheel_trans">
     <type>transmission_interface/SimpleTransmission</type>
     <joint name="${lr}_wheel_joint">
@@ -65,5 +67,5 @@
       <mechanicalReduction>50</mechanicalReduction>
     </actuator>
-  </transmission>
+  </transmission-->
 </macro>
 </robot>

File: robots/donatello/urdf/robot.xacro (robot description, xacro)
@@ -6,11 +6,11 @@
 <xacro:property name="chassisLength" value="0.16"/>
 <xacro:property name="chassisWidth" value="0.14"/>
-<xacro:property name="chassisMass" value="50"/>
+<xacro:property name="chassisMass" value="0.1"/>
 <xacro:property name="casterRadius" value="0.025"/>
-<xacro:property name="casterMass" value="5"/>
+<xacro:property name="casterMass" value="0.005"/>
 <xacro:property name="wheelWidth" value="0.015"/>
 <xacro:property name="wheelRadius" value="0.05"/>
 <xacro:property name="wheelPos" value="0.015"/>
-<xacro:property name="wheelMass" value="5"/>
+<xacro:property name="wheelMass" value="0.02"/>
 <xacro:property name="scanHeight" value="0.05"/>
 <xacro:property name="scanPos" value="0.015"/>
@@ -19,7 +19,7 @@
 <xacro:include filename="$(find roberta_sim)/robots/donatello/urdf/materials.xacro" />
 <xacro:include filename="$(find roberta_sim)/robots/donatello/urdf/macros.xacro" />
-<link name="footprint" />
+<link name="base_footprint" />
 <joint name="base_joint" type="fixed">
-  <parent link="footprint"/>
+  <parent link="base_footprint"/>
   <child link="chassis"/>
 </joint>
@@ -52,5 +52,5 @@
     <origin xyz="${casterRadius-chassisLength/2} 0 ${casterRadius-chassisHeight+wheelRadius}" rpy="0 0 0"/>
     <geometry>
-      <box size="${casterRadius*2} ${casterRadius*2} ${casterRadius*2}"/>
+      <sphere radius="${casterRadius}"/>
     </geometry>
   </collision>

Commit message: update burger maze

File: robots/donatello/urdf/macros.xacro (robot description, xacro)
@@ -55,17 +55,5 @@
   <origin xyz="${chassisLength/2-wheelPos} ${tY*wheelWidth/2+tY*chassisWidth/2} ${wheelRadius}" rpy="0 0 0" />
   <axis xyz="0 1 0" rpy="0 0 0" />
-  <!--limit effort="100" velocity="100"/>
-  <dynamics damping="0.0" friction="0.0"/-->
 </joint>
-<!--transmission name="${lr}_wheel_trans">
-    <type>transmission_interface/SimpleTransmission</type>
-    <joint name="${lr}_wheel_joint">
-      <hardwareInterface>hardware_interface/VelocityJointInterface</hardwareInterface>
-    </joint>
-    <actuator name="${lr}_wheel_motor">
-      <hardwareInterface>hardware_interface/VelocityJointInterface</hardwareInterface>
-      <mechanicalReduction>50</mechanicalReduction>
-    </actuator>
-  </transmission-->
 </macro>
 </robot>

File: robots/donatello/urdf/robot.xacro (robot description, xacro)
@@ -6,5 +6,5 @@
 <xacro:property name="chassisLength" value="0.16"/>
 <xacro:property name="chassisWidth" value="0.14"/>
-<xacro:property name="chassisMass" value="0.1"/>
+<xacro:property name="chassisMass" value="0.15"/>
 <xacro:property name="casterRadius" value="0.025"/>
 <xacro:property name="casterMass" value="0.005"/>
